Commit message: Updated urdf with swapping of left and right eye and changing axis for tilt
Signed-off-by: jpmnieles <jpmnieles@connect.ust.hk>

File: robot.urdf (robot description, URDF)
Before this commit: robot robot, 13 links, 12 joints
Joints:
- joint eyes_pitch: axis 0 1 0 -> 0 -1 0
- joint lefteye_yaw: origin xyz=0 -0.03 0 -> xyz=0 0.03 0
- joint righteye_yaw: origin xyz=0 0.03 0 -> xyz=0 -0.03 0

Commit message: Changed the urdf neck pitch axis
Signed-off-by: jpmnieles <jpmnieles@connect.ust.hk>

File: robot.urdf (robot description, URDF)
Before this commit: robot robot, 13 links, 12 joints
Joints:
- joint neck_pitch: axis 0 1 0 -> 0 -1 0
